Commit message: Checkpoint

File: newton/examples/assets/assets/urdf/franka_description/robots/franka_panda_gripper.urdf (robot description, URDF)
Before this commit: robot panda, 17 links, 16 joints
Joints:
- joint cam: origin xyz=0.03 0 0.05 rpy=3.14159265359 0 0 -> xyz=0.03 0 0.0587 rpy=3.14159265359 0 0
- joint panda_finger_joint2: axis 0 -1 0 -> (none); limit lower=0.0 upper=0.04 effort=20 velocity=0.2 -> (none); mimic joint=panda_finger_joint1 -> (none); type prismatic -> fixed

Commit message: Checkpoint

File: newton/examples/assets/assets/urdf/franka_description/robots/franka_panda_gripper.urdf (robot description, URDF)
Before this commit: robot panda, 17 links, 16 joints
Links:
- link panda_leftfinger: geometry collision box size=0.040 0.040 0.122; collision mesh filename=../../../umi/soft_gripper_finger.stl
- link panda_rightfinger: geometry collision box size=0.040 0.040 0.122; collision mesh filename=../../../umi/soft_gripper_finger.stl
Joints:
- joint panda_finger_joint2: axis (none) -> 0 -1 0; limit (none) -> lower=0.0 upper=0.04 effort=20 velocity=0.2; type fixed -> prismatic

Commit message: Fixed URDF

File: newton/examples/assets/assets/urdf/franka_description/robots/franka_panda_gripper.urdf (robot description, URDF)
Before this commit: robot panda, 17 links, 16 joints
Links:
- link panda_leftfinger: geometry collision box size=0.040 0.03 0.122; collision mesh filename=../../../umi/soft_gripper_finger.stl
- link panda_rightfinger: geometry collision box size=0.040 0.030 0.122; collision mesh filename=../../../umi/soft_gripper_finger.stl
Joints:
- joint panda_grip_vis_joint: origin xyz=0 0 0.1025 rpy=0 0 0 -> xyz=0 0 0.208 rpy=0 0 0
